Commit message: Fixed issues with mesh files. Sim appears to be running without error and is ready for testing.

File: src/m3pro_description/urdf/m3pro.urdf (robot description, URDF)
Before this commit: robot m3pro, 17 links, 16 joints
Links:
- link arm1: geometry visual mesh filename=package://m3pro_description/meshes/arm1.stl
- link arm2: geometry visual mesh filename=package://m3pro_description/meshes/arm2.stl
- link arm3: geometry visual mesh filename=package://m3pro_description/meshes/arm3.stl
- link arm4: geometry visual mesh filename=package://m3pro_description/meshes/arm4.stl
- link arm5: geometry visual mesh filename=package://m3pro_description/meshes/arm5.stl
- link arm_base_link: geometry visual mesh filename=package://m3pro_description/meshes/arm_base_Link.stl
- link base_link: geometry collision box size=0.24 0.18 0.12; visual mesh filename=package://m3pro_description/meshes/base_link.stl
- link camera_link: geometry visual mesh filename=package://m3pro_description/meshes/Camera.stl
- link gripper_link: geometry visual mesh filename=package://m3pro_description/meshes/Gripping.stl
- link lwheel1: geometry collision cylinder length=0.055 radius=0.04; visual mesh filename=package://m3pro_description/meshes/lwheel1.stl
- link lwheel2: geometry collision cylinder length=0.055 radius=0.04; visual mesh filename=package://m3pro_description/meshes/lwheel2.stl
- link rwheel1: geometry collision cylinder length=0.055 radius=0.04; visual mesh filename=package://m3pro_description/meshes/rwheel1.stl
- link rwheel2: geometry collision cylinder length=0.055 radius=0.04; visual mesh filename=package://m3pro_description/meshes/rwheel2.stl
