Commit message: Added missing bodies to URDF file. Also modified materials and colors of objects in the URDF that weren't showing up. All bodies now appear to be present in RVIZ.

File: src/m3pro_description/urdf/m3pro.urdf (robot description, URDF)
Before this commit: robot m3pro, 17 links, 16 joints
Links:
- removed link gripper_link
- added link gripping_housing, mass 0.012; visual mesh filename=package://m3pro_description/meshes/Gripping.stl
- added link llink1, mass 0.00427; visual mesh filename=package://m3pro_description/meshes/llink1.stl
- added link llink2, mass 0.00614; visual mesh filename=package://m3pro_description/meshes/llink2.stl
- added link llink3, mass 0.00271; visual mesh filename=package://m3pro_description/meshes/llink3.stl
- added link rlink1, mass 0.00470; visual mesh filename=package://m3pro_description/meshes/rlink1.stl
- added link rlink2, mass 0.00614; visual mesh filename=package://m3pro_description/meshes/rlink2.stl
- added link rlink3, mass 0.00271; visual mesh filename=package://m3pro_description/meshes/rlink3.stl
- added link wrist_camera_link; visual mesh filename=package://m3pro_description/meshes/DCW2.stl
Joints:
- added joint gripping_housing_joint: type fixed, parent arm5, child gripping_housing, origin xyz=-0.000625 0.00024 0.093235 rpy=3.108257 -1.570792 -3.108286
- added joint llink1_joint: type continuous, parent arm5, child llink1, origin xyz=-0.0044997 0.012375 0.029275 rpy=-1.570799 -0.603181 1.570799, axis 0 0 1, mimic joint=rlink1_joint multiplier=1.0 offset=0.0
- added joint llink2_joint: type continuous, parent llink1, child llink2, origin xyz=0.03 0 0.00125 rpy=0 0 -0.96762, axis 0 0 1, mimic joint=rlink1_joint multiplier=-1.0 offset=0.0
- added joint llink3_joint: type continuous, parent arm5, child llink3, origin xyz=-0.0044999 0.0045001 0.047275 rpy=-1.570799 -0.615160 1.570799, axis 0 0 1, mimic joint=rlink1_joint multiplier=1.0 offset=0.0
- added joint rlink2_joint: type continuous, parent rlink1, child rlink2, origin xyz=0.03 0 0.001 rpy=0 0 0.9667, axis 0 0 1, mimic joint=rlink1_joint multiplier=1.0 offset=0.0
- added joint rlink3_joint: type continuous, parent arm5, child rlink3, origin xyz=-0.0045001 -0.0044999 0.047275 rpy=1.570799 -0.612611 -1.570799, axis 0 0 1, mimic joint=rlink1_joint multiplier=-1.0 offset=0.0
- added joint wrist_camera_joint: type fixed, parent arm4, child wrist_camera_link, origin xyz=-0.0484 0.00245 0.0672 rpy=0.028287 -1.570796 0
- joint rlink1_joint: child gripper_link -> rlink1; origin xyz=-0.0048 -0.0126 0.029275 rpy=1.5708 -0.604 -1.5708 -> xyz=-0.0047503 -0.012625 0.029275 rpy=1.570801 -0.604091 -1.570801
